Commit message: Update cit_bldg2_19f

File: raspimouse_gazebo/materials/cit_bldg2_19f.world.xacro (robot description, xacro)
@@ -36,125 +36,83 @@
   </gui>
    <!-- horizontal -->
-  <xacro:wall>
+  <xacro:wall_corridor>
+    <pose> -9.76 1.145 0.25 0 0 1.57</pose>
+  </xacro:wall_corridor>
+  <xacro:wall_corridor>
+    <pose> -9.0 1.145 0.25 0 0 1.57</pose>
+  </xacro:wall_corridor>
+  <xacro:wall_corridor>
+    <pose> -7.0 1.145 0.25 0 0 1.57</pose>
+  </xacro:wall_corridor>
+  <xacro:wall_corridor>
+    <pose> -5.0 1.145 0.25 0 0 1.57</pose>
+  </xacro:wall_corridor>
+  <xacro:wall_corridor>
+    <pose> -3.0 1.145 0.25 0 0 1.57</pose>
+  </xacro:wall_corridor>
+  <xacro:wall_corridor>
     <pose> -1.0 1.145 0.25 0 0 1.57</pose>
-  </xacro:wall>
-  <xacro:wall>
-    <pose> -0.5 1.145 0.25 0 0 1.57</pose>
-  </xacro:wall>
-  <xacro:wall>
-    <pose> 0.0 1.145 0.25 0 0 1.57</pose>
-  </xacro:wall>
-  <xacro:wall>
-    <pose> 0.5 1.145 0.25 0 0 1.57</pose>
-  </xacro:wall>
-  <xacro:wall>
+  </xacro:wall_corridor>
+  <xacro:wall_corridor>
     <pose> 1.0 1.145 0.25 0 0 1.57</pose>
-  </xacro:wall>
-  <xacro:wall>
-    <pose> 1.5 1.145 0.25 0 0 1.57</pose>
-  </xacro:wall>
-  <xacro:wall>
-    <pose> 2.0 1.145 0.25 0 0 1.57</pose>
-  </xacro:wall>
+  </xacro:wall_corridor>
   <xacro:wall>
     <pose> 2.12 1.145 0.25 0 0 1.57</pose>
   </xacro:wall>
-  <xacro:wall>
-    <pose> 4.0 1.145 0.25 0 0 1.57</pose>
-  </xacro:wall>
-  <xacro:wall>
-    <pose> 4.5 1.145 0.25 0 0 1.57</pose>
-  </xacro:wall>
-  <xacro:wall>
-    <pose> 5.0 1.145 0.25 0 0 1.57</pose>
-  </xacro:wall>
-  <xacro:wall>
-    <pose> 5.5 1.145 0.25 0 0 1.57</pose>
-  </xacro:wall>
-  <xacro:wall>
-    <pose> 6.0 1.145 0.25 0 0 1.57</pose>
-  </xacro:wall>
-  <xacro:wall>
+  <xacro:wall_corridor>
+    <pose> 4.75 1.145 0.25 0 0 1.57</pose>
+  </xacro:wall_corridor>
+  <xacro:wall_corridor>
+    <pose> 6.75 1.145 0.25 0 0 1.57</pose>
+  </xacro:wall_corridor>
+  <xacro:wall>
+    <pose> 7.77 1.145 0.25 0 0 1.57</pose>
+  </xacro:wall>
+  <xacro:wall_corridor>
+    <pose> -15.0 -1.145 0.25 0 0 1.57</pose>
+  </xacro:wall_corridor>
+  <xacro:wall_corridor>
+    <pose> -13.0 -1.145 0.25 0 0 1.57</pose>
+  </xacro:wall_corridor>
+  <xacro:wall_corridor>
+    <pose> -11.0 -1.145 0.25 0 0 1.57</pose>
+  </xacro:wall_corridor>
+  <xacro:wall_corridor>
+    <pose> -9.0 -1.145 0.25 0 0 1.57</pose>
+  </xacro:wall_corridor>
+  <xacro:wall_corridor>
+    <pose> -7.0 -1.145 0.25 0 0 1.57</pose>
+  </xacro:wall_corridor>
+  <xacro:wall_corridor>
+    <pose> -5.0 -1.145 0.25 0 0 1.57</pose>
+  </xacro:wall_corridor>
+  <xacro:wall_corridor>
+    <pose> -3.0 -1.145 0.25 0 0 1.57</pose>
+  </xacro:wall_corridor>
+  <xacro:wall_corridor>
     <pose> -1.0 -1.145 0.25 0 0 1.57</pose>
-  </xacro:wall>
-  <xacro:wall>
-    <pose> -0.5 -1.145 0.25 0 0 1.57</pose>
-  </xacro:wall>
-  <xacro:wall>
-    <pose> 0.0 -1.145 0.25 0 0 1.57</pose>
-  </xacro:wall>
-  <xacro:wall>
-    <pose> 0.5 -1.1455 0.25 0 0 1.57</pose>
-  </xacro:wall>
-  <xacro:wall>
+  </xacro:wall_corridor>
+  <xacro:wall_corridor>
     <pose> 1.0 -1.1455 0.25 0 0 1.57</pose>
-  </xacro:wall>
-  <xacro:wall>
-    <pose> 1.5 -1.145 0.25 0 0 1.57</pose>
-  </xacro:wall>
-  <xacro:wall>
-    <pose> 2.0 -1.145 0.25 0 0 1.57</pose>
-  </xacro:wall>
-  <xacro:wall>
-    <pose> 2.5 -1.145 0.25 0 0 1.57</pose>
-  </xacro:wall>
-  <xacro:wall>
+  </xacro:wall_corridor>
+  <xacro:wall_corridor>
     <pose> 3.0 -1.145 0.25 0 0 1.57</pose>
-  </xacro:wall>
-  <xacro:wall>
-    <pose> 3.5 -1.145 0.25 0 0 1.57</pose>
-  </xacro:wall>
-  <xacro:wall>
-    <pose> 4.0 -1.145 0.25 0 0 1.57</pose>
-  </xacro:wall>
-  <xacro:wall>
-    <pose> 4.5 -1.145 0.25 0 0 1.57</pose>
-  </xacro:wall>
-  <xacro:wall>
+  </xacro:wall_corridor>
+  <xacro:wall_corridor>
     <pose> 5.0 -1.145 0.25 0 0 1.57</pose>
-  </xacro:wall>
-  <xacro:wall>
-    <pose> 5.5 -1.145 0.25 0 0 1.57</pose>
-  </xacro:wall>
-  <xacro:wall>
-    <pose> 6.0 -1.145 0.25 0 0 1.57</pose>
-  </xacro:wall>
+  </xacro:wall_corridor>
+  <xacro:wall_corridor>
+    <pose> 7.0 -1.145 0.25 0 0 1.57</pose>
+  </xacro:wall_corridor>
   <!-- vertical -->
-  <xacro:wall>
-    <pose> 2.32 1.345 0.25 0 0 0</pose>
-  </xacro:wall>
-  <xacro:wall>
-    <pose> 2.32 1.845 0.25 0 0 0</pose>
-  </xacro:wall>
-  <xacro:wall>
-    <pose> 2.32 2.345 0.25 0 0 0</pose>
-  </xacro:wall>
-  <xacro:wall>
-    <pose> 2.32 2.845 0.25 0 0 0</pose>
-  </xacro:wall>
-  <xacro:wall>
-    <pose> 2.32 3.345 0.25 0 0 0</pose>
-  </xacro:wall>
-  <xacro:wall>
-    <pose> 2.32 3.845 0.25 0 0 0</pose>
-  </xacro:wall>
-  <xacro:wall>
-    <pose> 2.32 4.345 0.25 0 0 0</pose>
-  </xacro:wall>
-  <xacro:wall>
-    <pose> 2.32 4.845 0.25 0 0 0</pose>
-  </xacro:wall>
-  <xacro:wall>
-    <pose> 2.32 5.345 0.25 0 0 0</pose>
-  </xacro:wall>
-  <xacro:wall>
-    <pose> 2.32 5.845 0.25 0 0 0</pose>
-  </xacro:wall>
-  <xacro:wall>
-    <pose> 2.32 6.345 0.25 0 0 0</pose>
-  </xacro:wall>
-  <xacro:wall>
-    <pose> 2.32 6.845 0.25 0 0 0</pose>
-  </xacro:wall>
+  <xacro:wall_corridor>
+    <pose> 2.32 2.095 0.25 0 0 0</pose>
+  </xacro:wall_corridor>
+  <xacro:wall_corridor>
+    <pose> 2.32 4.095 0.25 0 0 0</pose>
+  </xacro:wall_corridor>
+  <xacro:wall_corridor>
+    <pose> 2.32 6.095 0.25 0 0 0</pose>
+  </xacro:wall_corridor>
   <xacro:wall>
     <pose> 2.32 7.345 0.25 0 0 0</pose>
@@ -217,46 +175,191 @@
     <pose> 3.8 8.345 0.25 0 0 0</pose>
   </xacro:wall>
-  <xacro:wall>
-    <pose> 4.0 7.58 0.25 0 0 1.57</pose>
-  </xacro:wall>
-  <xacro:wall>
-    <pose> 4.5 7.58 0.25 0 0 1.57</pose>
+  <xacro:wall_corridor>
+    <pose> 4.75 7.58 0.25 0 0 1.57</pose>
+  </xacro:wall_corridor>
+  <xacro:wall_corridor>
+    <pose> 6.75 7.58 0.25 0 0 1.57</pose>
+  </xacro:wall_corridor>
+  <xacro:wall>
+    <pose> 7.82 7.58 0.25 0 0 1.57</pose>
+  </xacro:wall>
+  <xacro:wall_corridor>
+    <pose> 8.02 6.63 0.25 0 0 0</pose>
+  </xacro:wall_corridor>
+  <xacro:wall_corridor>
+    <pose> 8.02 4.63 0.25 0 0 0</pose>
+  </xacro:wall_corridor>
+  <xacro:wall_corridor>
+    <pose> 8.02 2.63 0.25 0 0 0</pose>
+  </xacro:wall_corridor>
+  <xacro:wall>
+    <pose> 8.02 1.395 0.25 0 0 0</pose>
   </xacro:wall>
   <!-- horizontal -->
-  <xacro:wall>
-    <pose> 4.0 8.545 0.25 0 0 1.57</pose>
-  </xacro:wall>
-  <xacro:wall>
-    <pose> 4.5 8.545 0.25 0 0 1.57</pose>
-  </xacro:wall>
-  <xacro:wall>
-    <pose> 5.0 8.545 0.25 0 0 1.57</pose>
-  </xacro:wall>
-  <xacro:wall>
-    <pose> 5.5 8.545 0.25 0 0 1.57</pose>
-  </xacro:wall>
-  <xacro:wall>
-    <pose> 6.0 8.545 0.25 0 0 1.57</pose>
-  </xacro:wall>
-  <xacro:wall>
-    <pose> 2.12 8.545 0.25 0 0 1.57</pose>
-  </xacro:wall>
-  <xacro:wall>
-    <pose> 1.62 8.545 0.25 0 0 1.57</pose>
-  </xacro:wall>
-  <xacro:wall>
-    <pose> 1.12 8.545 0.25 0 0 1.57</pose>
-  </xacro:wall>
-  <xacro:wall>
-    <pose> 0.62 8.545 0.25 0 0 1.57</pose>
-  </xacro:wall>
-  <xacro:wall>
-    <pose> 0.12 8.545 0.25 0 0 1.57</pose>
-  </xacro:wall>
-  <xacro:wall>
-    <pose> -0.38 8.545 0.25 0 0 1.57</pose>
-  </xacro:wall>
-  <xacro:wall>
-    <pose> -0.88 8.545 0.25 0 0 1.57</pose>
+  <xacro:wall_corridor>
+    <pose> 4.75 8.545 0.25 0 0 1.57</pose>
+  </xacro:wall_corridor>
+  <xacro:wall_corridor>
+    <pose> 6.75 8.545 0.25 0 0 1.57</pose>
+  </xacro:wall_corridor>
+  <xacro:wall_corridor>
+    <pose> 1.37 8.545 0.25 0 0 1.57</pose>
+  </xacro:wall_corridor>
+  <xacro:wall_corridor>
+    <pose> -0.63 8.545 0.25 0 0 1.57</pose>
+  </xacro:wall_corridor>
+  <xacro:wall_corridor>
+    <pose> -2.63 8.545 0.25 0 0 1.57</pose>
+  </xacro:wall_corridor>
+  <xacro:wall_corridor>
+    <pose> -4.63 8.545 0.25 0 0 1.57</pose>
+  </xacro:wall_corridor>
+  <xacro:wall_corridor>
+    <pose> -6.63 8.545 0.25 0 0 1.57</pose>
+  </xacro:wall_corridor>
+  <xacro:wall_corridor>
+    <pose> -8.44 8.545 0.25 0 0 1.57</pose>
+  </xacro:wall_corridor>
+ <xacro:wall_corridor>
+    <pose> -12.60 8.545 0.25 0 0 1.57</pose>
+  </xacro:wall_corridor>
+  <xacro:wall_corridor>
+    <pose> -14.60 8.545 0.25 0 0 1.57</pose>
+  </xacro:wall_corridor>
+  <xacro:wall_corridor>
+    <pose> -15.88 10.545 0.25 0 0 1.57</pose>
+  </xacro:wall_corridor>
+  <xacro:wall_corridor>
+    <pose> -13.88 10.545 0.25 0 0 1.57</pose>
+  </xacro:wall_corridor>
+  <xacro:wall_corridor>
+    <pose> -11.88 10.545 0.25 0 0 1.57</pose>
+  </xacro:wall_corridor>
+  <xacro:wall_corridor>
+    <pose> -9.88 10.545 0.25 0 0 1.57</pose>
+  </xacro:wall_corridor>
+  <xacro:wall_corridor>
+    <pose> -7.88 10.545 0.25 0 0 1.57</pose>
+  </xacro:wall_corridor>
+  <xacro:wall_corridor>
+    <pose> -5.88 10.545 0.25 0 0 1.57</pose>
+  </xacro:wall_corridor>
+  <xacro:wall_corridor>
+    <pose> -3.88 10.545 0.25 0 0 1.57</pose>
+  </xacro:wall_corridor>
+  <xacro:wall_corridor>
+    <pose> -1.88 10.545 0.25 0 0 1.57</pose>
+  </xacro:wall_corridor>
+  <xacro:wall_corridor>
+    <pose> 0.12 10.545 0.25 0 0 1.57</pose>
+  </xacro:wall_corridor>
+  <xacro:wall_corridor>
+    <pose> 2.12 10.545 0.25 0 0 1.57</pose>
+  </xacro:wall_corridor>
+  <xacro:wall_corridor>
+    <pose> 4.12 10.545 0.25 0 0 1.57</pose>
+  </xacro:wall_corridor>
+  <xacro:wall_corridor>
+    <pose> 6.12 10.545 0.25 0 0 1.57</pose>
+  </xacro:wall_corridor>
+  <xacro:wall_corridor>
+    <pose> 7.12 10.545 0.25 0 0 1.57</pose>
+  </xacro:wall_corridor>
+  <!-- vertical -->
+  <xacro:wall_corridor>
+    <pose> -9.39 7.595 0.25 0 0 0</pose>
+  </xacro:wall_corridor>
+  <xacro:wall>
+    <pose> -9.39 6.345 0.25 0 0 0</pose>
+  </xacro:wall>
+  <xacro:wall>
+    <pose> -9.39 5.845 0.25 0 0 0</pose>
+  </xacro:wall>
+  <xacro:wall>
+    <pose> -9.59 5.645 0.25 0 0 1.57</pose>
+  </xacro:wall>
+  <xacro:wall>
+    <pose> -10.09 5.645 0.25 0 0 1.57</pose>
+  </xacro:wall>
+  <xacro:wall>
+    <pose> -10.56 5.645 0.25 0 0 1.57</pose>
+  </xacro:wall>
+  <xacro:wall_corridor>
+    <pose> -10.76 4.695 0.25 0 0 0</pose>
+  </xacro:wall_corridor>
+  <xacro:wall_corridor>
+    <pose> -10.76 2.695 0.25 0 0 0</pose>
+  </xacro:wall_corridor>
+  <xacro:wall_corridor>
+    <pose> -10.76 2.095 0.25 0 0 0</pose>
+  </xacro:wall_corridor>
+  <xacro:wall_corridor>
+    <pose> -12.66 1.145 0.25 0 0 1.57</pose>
+  </xacro:wall_corridor>
+  <xacro:wall_corridor>
+    <pose> -14.66 1.145 0.25 0 0 1.57</pose>
+  </xacro:wall_corridor>
+  <xacro:wall>
+    <pose> -15.7 1.145 0.25 0 0 1.57</pose>
+  </xacro:wall>
+  <xacro:wall>
+    <pose> -11.71 1.345 0.25 0 0 0</pose>
+  </xacro:wall>
+  <xacro:wall>
+    <pose> -11.71 1.845 0.25 0 0 0</pose>
+  </xacro:wall>
+  <xacro:wall>
+    <pose> -11.71 1.915 0.25 0 0 0</pose>
+  </xacro:wall>
+  <xacro:wall>
+    <pose> -11.91 2.115 0.25 0 0 1.57</pose>
+  </xacro:wall>
+  <xacro:wall>
+    <pose> -12.41 2.115 0.25 0 0 1.57</pose>
+  </xacro:wall>
+  <xacro:wall_corridor>
+    <pose> -12.61 3.065 0.25 0 0 0</pose>
+  </xacro:wall_corridor>
+  <xacro:wall_corridor>
+    <pose> -12.61 5.065 0.25 0 0 0</pose>
+  </xacro:wall_corridor>
+  <xacro:wall_corridor>
+    <pose> -12.61 5.215 0.25 0 0 0</pose>
+  </xacro:wall_corridor>
+  <xacro:wall>
+    <pose> -12.41 7.565 0.25 0 0 1.57</pose>
+  </xacro:wall>
+  <xacro:wall>
+    <pose> -11.91 7.565 0.25 0 0 1.57</pose>
+  </xacro:wall>
+  <xacro:wall>
+    <pose> -11.85 7.565 0.25 0 0 1.57</pose>
+  </xacro:wall>
+  <xacro:wall_corridor>
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
File: raspimouse_gazebo/materials/sample_maze.wall.xacro (robot description, xacro)
@@ -58,3 +58,60 @@
     </model>
   </xacro:macro>
+  <xacro:macro name="wall_corridor" params="*pose">
+    <model name='wall_corridor'>
+      <!-- <pose>&#45;0.09 0 0.5 0 0 1.57</pose> -->
+      <insert_block name="pose"/>
+      <link name='link'>
+        <inertial>
+          <mass>10</mass>
+          <inertia>
+            <ixx>1</ixx>
+            <ixy>0</ixy>
+            <ixz>0</ixz>
+            <iyy>1</iyy>
+            <iyz>0</iyz>
+            <izz>1</izz>
+          </inertia>
+        </inertial>
+        <collision name='collision'>
+          <geometry>
+            <box>
+              <size>0.1 2.0 0.5</size>
+            </box>
+          </geometry>
+          <max_contacts>10</max_contacts>
+          <surface>
+            <bounce/>
+            <friction>
+              <ode/>
+            </friction>
+            <contact>
+              <ode/>
+            </contact>
+          </surface>
+        </collision>
+        <visual name='visual'>
+          <geometry>
+            <box>
+              <size>0.1 2.0 0.5</size>
+            </box>
+          </geometry>
+          <material>
+            <script>
+              <uri>file://media/materials/scripts/gazebo.material</uri>
+              <name>Gazebo/White</name>
+            </script>
+          </material>
+        </visual>
+        <velocity_decay>
+          <linear>0</linear>
+          <angular>0</angular>
+        </velocity_decay>
+        <self_collide>0</self_collide>
+        <kinematic>0</kinematic>
+        <gravity>1</gravity>
+      </link>
+      <static>1</static>
+    </model>
+  </xacro:macro>
 </sdf>
